File: new/list2.kicad_sch (KiCad schematic)
At the start: 9 parts, among them J1 Conn_01x20_Male, J7 Conn_01x02_Male, J8 Conn_01x05_Male, J9 Conn_01x04_Male

Commit message: ..
Other:
- note added: "5 200 руб. 5V, 3А 60x94 мм"
- note added: "HDMI + USB-C"
- note removed: "5 200 руб."
- note removed: "HDMI"
Changed lines of the file:
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@@
-(kicad_sch (version 20230121) (generator eeschema)
+(kicad_sch (version 20230409) (generator eeschema)
   (paper "A4")
   (title_block
@@
     (fill (type none))
   )
-  (text "  Микро-\n компьютер \nOrange PI 3 \nLTS 2GB 8GB" (at 229.87 53.34 0)
+  (text "  Микро-\n компьютер \nOrange PI 3 \nLTS 2GB 8GB" (exclude_from_sim no)
+ (at 229.87 53.34 0)
     (effects (font (size 4 4)) (justify left bottom))
   )
-  (text "HDMI" (at 233.68 96.52 0)
+  (text "HDMI + USB-C" (exclude_from_sim no)
+ (at 233.68 99.06 0)
     (effects (font (size 3 3) bold) (justify left bottom))
   )
-  (text "RS-485\nUART-RS485, RJ-45 (Trema-модуль V2.0)\nвроде без гальваническо развязки"
+  (text "RS-485\nUART-RS485, RJ-45 (Trema-модуль V2.0)\nвроде без гальваническо развязки" (exclude_from_sim no)
     (at 119.38 21.59 0)
     (effects (font (size 1.27 1.27)) (justify left bottom))
   )
-  (text "Вариант с микро пк." (at 210.82 153.67 0)
+  (text "Вариант с микро пк." (exclude_from_sim no)
+ (at 210.82 153.67 0)
     (effects (font (size 4 4) bold) (justify left bottom))
   )
-  (text "STM32 Smart V2.0" (at 58.42 105.41 0)
+  (text "STM32 Smart V2.0" (exclude_from_sim no)
+ (at 58.42 105.41 0)
     (effects (font (size 2 2)) (justify left bottom))
   )
-  (text "RS485" (at 208.28 21.59 0)
+  (text "RS485" (exclude_from_sim no)
+ (at 208.28 21.59 0)
     (effects (font (size 1.27 1.27) bold) (justify left bottom))
   )
-  (text "5 200 руб." (at 238.76 82.55 0)
+  (text "5 200 руб.\n5V, 3А\n60x94 мм" (exclude_from_sim no)
+ (at 245.11 91.44 0)
     (effects (font (size 3 3) bold) (justify left bottom))
   )
-  (text "кнопки ввода" (at 105.41 153.67 0)
+  (text "кнопки ввода" (exclude_from_sim no)
+ (at 105.41 153.67 0)
     (effects (font (size 4 4)) (justify left bottom))
   )
-  (text "   плата\nc дисплеем\n  HD44780" (at 148.59 95.25 0)
+  (text "   плата\nc дисплеем\n  HD44780" (exclude_from_sim no)
+ (at 148.59 95.25 0)
     (effects (font (size 4 4)) (justify left bottom))
   )
-  (text "7-дюймовый\n сенсорный \n экран\n ссылка" (at 229.87 133.35 0)
+  (text "7-дюймовый\n сенсорный \n экран\n ссылка" (exclude_from_sim no)
+ (at 229.87 133.35 0)
     (effects (font (size 4 4)) (justify left bottom) (href "https://www.avito.ru/moskva/tovary_dlya_kompyutera/7-dyuymovyy_sensornyy_ekran_s_chehlom_dlya_mikrokomp_3228330568?slocation=621540"))
   )
-  (text "5 100 руб." (at 241.3 140.97 0)
+  (text "5 100 руб." (exclude_from_sim no)
+ (at 241.3 140.97 0)
     (effects (font (size 3 3) bold) (justify left bottom))
   )
-  (text "UART" (at 118.11 64.77 0)
+  (text "UART" (exclude_from_sim no)
+ (at 118.11 64.77 0)
     (effects (font (size 3 3) bold) (justify left bottom))
   )
-  (text "   плата\nуправления" (at 54.61 96.52 0)
+  (text "   плата\nуправления" (exclude_from_sim no)
+ (at 54.61 96.52 0)
     (effects (font (size 4 4)) (justify left bottom))
   )
@@
       (effects (font (size 1.27 1.27)) hide)
     )
+    (pin "1")
+    (pin "2")
+    (pin "3")
+    (pin "4")
     (pin "5")
-    (pin "1")
-    (pin "2")
-    (pin "4")
-    (pin "3")
     (instances
       (project "new"
@@
       (effects (font (size 1.27 1.27)) hide)
     )
+    (pin "1")
+    (pin "2")
+    (pin "3")
+    (pin "4")
     (pin "5")
-    (pin "1")
-    (pin "2")
-    (pin "4")
-    (pin "3")
     (instances
       (project "new"
@@
       (effects (font (size 1.27 1.27)) hide)
     )
+    (pin "1")
+    (pin "2")
+    (pin "3")
+    (pin "4")
     (pin "5")
-    (pin "1")
-    (pin "2")
-    (pin "4")
-    (pin "3")
     (instances
       (project "new"
@@
       (effects (font (size 1.27 1.27)) hide)
     )
+    (pin "1")
+    (pin "10")
+    (pin "11")
+    (pin "12")
+    (pin "13")
+    (pin "14")
+    (pin "15")
+    (pin "16")
+    (pin "17")
     (pin "18")
-    (pin "2")
-    (pin "4")
+    (pin "19")
+    (pin "2")
+    (pin "20")
+    (pin "3")
+    (pin "4")
+    (pin "5")
+    (pin "6")
+    (pin "7")
+    (pin "8")
+    (pin "9")
+    (instances
+      (project "new"
+        (path "/ef117e5f-52c6-4535-bb06-6f0bbe70a6e7"
+          (reference "J1") (unit 1)
+        )
+        (path "/ef117e5f-52c6-4535-bb06-6f0bbe70a6e7/dcd91f8f-6d85-40bc-b09c-b2de90179c16"
+          (reference "J6") (unit 1)
+        )
+      )
+    )
+  )
+  (symbol (lib_id "Connector:Conn_01x05_Male") (at 123.19 25.4 270) (unit 1)
+    (in_bom yes) (on_board yes) (dnp no)
+    (property "Reference" "J8" (at 113.03 26.67 90)
+      (effects (font (size 1.27 1.27)))
+    )
+    (property "Value" "Conn_01x05_Male" (at 130.81 26.035 0)
+      (effects (font (size 1.27 1.27)) hide)
+    )
+    (property "Footprint" "" (at 123.19 25.4 0)
+      (effects (font (size 1.27 1.27)) hide)
+    )
+    (property "Datasheet" "~" (at 123.19 25.4 0)
+      (effects (font (size 1.27 1.27)) hide)
+    )
+    (pin "1")
+    (pin "2")
+    (pin "3")
+    (pin "4")
+    (pin "5")
+    (instances
+      (project "new"
+        (path "/ef117e5f-52c6-4535-bb06-6f0bbe70a6e7"
+          (reference "J8") (unit 1)
+        )
+        (path "/ef117e5f-52c6-4535-bb06-6f0bbe70a6e7/dcd91f8f-6d85-40bc-b09c-b2de90179c16"
+          (reference "J11") (unit 1)
+        )
+      )
+    )
+  )
+  (symbol (lib_id "Connector:Conn_01x20_Male") (at 135.89 90.17 0) (unit 1)
+    (in_bom yes) (on_board yes) (dnp no)
+    (property "Reference" "J1" (at 134.62 64.77 0)
+      (effects (font (size 1.27 1.27)))
+    )
+    (property "Value" "Conn_01x20_Male" (at 136.525 64.77 0)
+      (effects (font (size 1.27 1.27)) hide)
+    )
+    (property "Footprint" "Connector_PinHeader_2.54mm:PinHeader_1x20_P2.54mm_Vertical" (at 135.89 90.17 0)
+      (effects (font (size 1.27 1.27)) hide)
+    )
+    (property "Datasheet" "~" (at 135.89 90.17 0)
+      (effects (font (size 1.27 1.27)) hide)
+    )
+    (pin "1")
+    (pin "10")
     (pin "11")
+    (pin "12")
+    (pin "13")
+    (pin "14")
+    (pin "15")
     (pin "16")
-    (pin "1")
-    (pin "14")
+    (pin "17")
+    (pin "18")
     (pin "19")
-    (pin "12")
+    (pin "2")
+    (pin "20")
+    (pin "3")
+    (pin "4")
     (pin "5")
+    (pin "6")
+    (pin "7")
     (pin "8")
-    (pin "15")
-    (pin "7")
     (pin "9")
-    (pin "6")
-    (pin "20")
-    (pin "10")
-    (pin "17")
-    (pin "13")
-    (pin "3")
-    (instances
-      (project "new"
-        (path "/ef117e5f-52c6-4535-bb06-6f0bbe70a6e7"
-          (reference "J1") (unit 1)
-        )
-        (path "/ef117e5f-52c6-4535-bb06-6f0bbe70a6e7/dcd91f8f-6d85-40bc-b09c-b2de90179c16"
-          (reference "J6") (unit 1)
-        )
-      )
-    )
-  )
-  (symbol (lib_id "Connector:Conn_01x05_Male") (at 123.19 25.4 270) (unit 1)
-    (in_bom yes) (on_board yes) (dnp no)
-    (property "Reference" "J8" (at 113.03 26.67 90)
-      (effects (font (size 1.27 1.27)))
-    )
-    (property "Value" "Conn_01x05_Male" (at 130.81 26.035 0)
-      (effects (font (size 1.27 1.27)) hide)
-    )
-    (property "Footprint" "" (at 123.19 25.4 0)
-      (effects (font (size 1.27 1.27)) hide)
-    )
-    (property "Datasheet" "~" (at 123.19 25.4 0)
-      (effects (font (size 1.27 1.27)) hide)
-    )
-    (pin "5")
-    (pin "1")
-    (pin "2")
-    (pin "4")
-    (pin "3")
-    (instances
-      (project "new"
-        (path "/ef117e5f-52c6-4535-bb06-6f0bbe70a6e7"
-          (reference "J8") (unit 1)
-        )
-        (path "/ef117e5f-52c6-4535-bb06-6f0bbe70a6e7/dcd91f8f-6d85-40bc-b09c-b2de90179c16"
-          (reference "J11") (unit 1)
-        )
-      )
-    )
-  )
-  (symbol (lib_id "Connector:Conn_01x20_Male") (at 135.89 90.17 0) (unit 1)
-    (in_bom yes) (on_board yes) (dnp no)
-    (property "Reference" "J1" (at 134.62 64.77 0)
-      (effects (font (size 1.27 1.27)))
-    )
-    (property "Value" "Conn_01x20_Male" (at 136.525 64.77 0)
-      (effects (font (size 1.27 1.27)) hide)
-    )
-    (property "Footprint" "Connector_PinHeader_2.54mm:PinHeader_1x20_P2.54mm_Vertical" (at 135.89 90.17 0)
-      (effects (font (size 1.27 1.27)) hide)
-    )
-    (property "Datasheet" "~" (at 135.89 90.17 0)
-      (effects (font (size 1.27 1.27)) hide)
-    )
-    (pin "18")
-    (pin "2")
-    (pin "4")
-    (pin "11")
-    (pin "16")
-    (pin "1")
-    (pin "14")
-    (pin "19")
-    (pin "12")
-    (pin "5")
-    (pin "8")
-    (pin "15")
-    (pin "7")
-    (pin "9")
-    (pin "6")
-    (pin "20")
-    (pin "10")
-    (pin "17")
-    (pin "13")
-    (pin "3")
     (instances
       (project "new"
@@
       (effects (font (size 1.27 1.27)) hide)
     )
-    (pin "2")
-    (pin "1")
+    (pin "1")
+    (pin "2")
     (instances
       (project "new"
@@
       (effects (font (size 1.27 1.27)) hide)
     )
-    (pin "2")
-    (pin "1")
-    (pin "4")
-    (pin "3")
+    (pin "1")
+    (pin "2")
+    (pin "3")
+    (pin "4")
     (instances
       (project "new"
@@
       (effects (font (size 1.27 1.27)) hide)
     )
-    (pin "2")
-    (pin "1")
-    (instances
-      (project "new"
+    (pin "1")
+    (pin "2")
+    (instances
+      (project "new"
