File: new/new.kicad_sch (KiCad schematic)
At the start: 36 parts, among them J1 Conn_01x20_Male, J10 Conn_01x04_Male, J2 Conn_01x04_Male, J3 Conn_01x04_Male, J4 Conn_01x04_Male, J5 Conn_01x04_Male, J7 Conn_01x02_Male, J8 Conn_01x05_Male, J9 Conn_01x04_Male, K1 RSM822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

Commit message: ..
Parts:
- removed K1, K2: RSM822, Relay_THT:Relay_DPDT_Finder_40.52, symbol Relay:RSM822
- added BZ2: Buzzer, symbol Device:Buzzer
- added C1: C, symbol Device:C
- added D8: DIODE, symbol pspice:DIODE
- added J19: Conn_01x02_Male, symbol Connector:Conn_01x02_Male
- added K1: NT90TP-NCE-DC12V-CB-0.9, symbol Relay:Relay_SPDT
- added K3 (x2): T73 12VDC (833H) 10A, symbol Relay:Relay_SPDT
- added L1, L2: L, symbol Device:L
- added Q3: 2N7002, Package_TO_SOT_SMD:SOT-23, symbol Transistor_FET:2N7002
- added R10, R11, R12, R13: R, symbol Device:R
- added SW4: SW_Push, symbol Switch:SW_Push
- added U3: EL817, Package_DIP:DIP-4_W7.62mm, symbol Isolator:EL817
- AC-DC: value AC-DC 85-265V выход 12V 0.45A 5W -> IRM-30-12ST, AC/DC преобразователь, 12В,2.5А,30Вт
Connections:
- net +12V: now also D1.2 (A), D2.2 (A), D6.2 (A), D7.2 (A), BZ2.1 (-), D8.2 (A), K1.A1, K3.A1, K3.A1
- net +5V: no longer D1.2 (A), D2.2 (A)
- net GND: now also BZ2.2 (+), C1.2, Q3.2 (S), R13.1, SW4.1, U3.3
- net GNDD: now also U3.2
- net at D2.1 (K), Q1.3 (D), SW3.2: now also R9.2, K3.A2, K3.A2
- net at J3.2 (Pin_2): now also K3.14, K3.14; no longer R9.2
- net at R5.2: now also D1.1 (K), Q2.3 (D), SW2.2, K1.A2; no longer J2.2 (Pin_2)
- net at AC-DC.5 (AC/L), AC-DC1.5 (AC/L), J10.2 (Pin_2)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: now also K1.11, K3.11, K3.11
- net at AC-DC.1 (AC/N), AC-DC1.1 (AC/N), J10.3 (Pin_3)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: now also J2.1 (Pin_1), J3.1 (Pin_1)
- net at J1.17 (Pin_17): now also R10.1
- net at SW1.1: now also L2.2
- net at SW1.3: now also J19.2 (Pin_2)
- new net: D8.1 (K), Q3.3 (D), SW4.2
- new net: J2.2 (Pin_2), K1.14
- new net: C1.1, L1.2, R11.1, R12.1, R13.2
- new net: R10.2, U3.1
- new net: Q3.1 (G), U3.4
- new net: L1.1, R11.2
- new net: K3.12, K3.12
- new net: J19.1 (Pin_1), L2.1
- new net +3.3V: R12.2
Other:
- note added: "SCT-013"
- note added: "in - 0.9 W"
- note added: "Зуммер"
- note added: "измеритель тока"
- moved on the sheet: AC-DC, AC-DC1, D1, D2, D3, D4, D5, D6, D7, J1, J10, J2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
